Commit message: Initial joint states.

File: urdf/braccio.urdf (robot description, URDF)
Before this commit: robot visual, 9 links, 8 joints
Joints:
- joint base: limit lower=0.0 upper=3.141592653589793 effort=1000.0 velocity=0.5 -> lower=0.0 upper=3.141592653589793 effort=1000.0 velocity=4.0
- joint elbow: limit lower=0 upper=3.141592653589793 effort=1000.0 velocity=0.5 -> lower=0 upper=3.141592653589793 effort=1000.0 velocity=4.0
- joint shoulder: limit lower=0.2617993877991494 upper=2.8797932657906435 effort=1000.0 velocity=0.5 -> lower=0.2617993877991494 upper=2.8797932657906435 effort=1000.0 velocity=4.0
- joint wrist_pitch: limit lower=0 upper=3.141592653589793 effort=1000.0 velocity=0.5 -> lower=0 upper=3.141592653589793 effort=1000.0 velocity=4.0
- joint wrist_roll: limit lower=0.0 upper=3.141592653589793 effort=1000.0 velocity=0.5 -> lower=0.0 upper=3.141592653589793 effort=1000.0 velocity=4.0

Commit message: Improved gripper model.

File: urdf/braccio.urdf (robot description, URDF)
Before this commit: robot visual, 9 links, 8 joints
Links:
- removed link gripper_left
- removed link gripper_right
- added link gripper_fix; visual mesh filename=package://braccio_description/meshes/gripper_fix.stl
- added link gripper_movable; visual mesh filename=package://braccio_description/meshes/gripper_movable.stl
Joints:
- removed joint gripper_left
- removed joint gripper_right
- added joint gripper_fix: type fixed, parent gripper_base, child gripper_fix, origin xyz=0 0.0 0.007 rpy=0 0 0
- added joint gripper_movable: type revolute, parent gripper_base, child gripper_movable, origin xyz=0.01559 0 0.007 rpy=0 0 0, axis 0 -1 0, limit lower=0.17453292519943295 upper=1.2740903539558606 effort=1000.0 velocity=4.0
